Commit message: Fix car_4w.urdf wheels floating: visual radius 0.32 -> 0.358 to match physics
The preset car_4w_rwd_ackermann imposes a 0.358 m physics wheel radius
(_hjw_wheel_overrides, matching the HJW/golden_JMK reference), but car_4w.urdf
drew the visual cylinder at radius 0.32 m. The raycast suspension rests the
chassis for a 0.358 m wheel, so the smaller visual wheel floated ~38 mm above
the contact point -- visible as wheels hovering over the surface in
terrain_drive --viewer. Set the four wheel visuals to radius 0.358 (pure visual
change; physics already used 0.358). 96 pytest pass; terrain_drive/quickstart
drive identically. Bump 1.0.5 -> 1.0.6.

File: samples/urdf/car_4w.urdf (robot description, URDF)
Before this commit: robot car_4w, 11 links, 10 joints
Links:
- link front_left_wheel: geometry visual cylinder length=0.20 radius=0.358
- link front_right_wheel: geometry visual cylinder length=0.20 radius=0.358
- link rear_left_wheel: geometry visual cylinder length=0.20 radius=0.358
- link rear_right_wheel: geometry visual cylinder length=0.20 radius=0.358
